Commit message: Seperate Armcontrol and printing

File: src/youbot_print/resource/cube.urdf (robot description, URDF)
Before this commit: robot cube, 1 links, 0 joints
Links:
- link box: mass None -> 0.01; geometry collision sphere radius=0.1; visual sphere radius=0.1

Commit message: Second version of printing

File: src/youbot_print/resource/cube.urdf (robot description, URDF)
Before this commit: robot cube, 1 links, 0 joints
Links:
- link box: geometry collision box size=0.01 0.01 0.01; visual box size=0.01 0.01 0.01
